Commit message: changes

File: src/diffdrive_arduino/description/urdf/diffbot.urdf.xacro (robot description, xacro)
@@ -9,5 +9,5 @@
   <xacro:include filename="$(find diffdrive_arduino)/ros2_control/diffbot.ros2_control.xacro" />
   <xacro:include filename="inertial_macros.xacro"/>
-  <xacro:include filename="lidar2.xacro" />
+  <xacro:include filename="lidar.xacro" />
   <xacro:diffbot prefix="$(arg prefix)" />
   <xacro:diffbot_ros2_control

File: src/diffdrive_arduino/description/urdf/lidar.xacro (robot description, xacro)
@@ -3,5 +3,5 @@
     <joint name="laser_joint" type="fixed">
         <origin xyz="0.031539 -0.0015685 0.20" rpy="0 0 0" />
-        <parent link="chassis" />
+        <parent link="base_link" />
         <child link="laser_frame" />
     </joint>
@@ -16,5 +16,5 @@
           </visual>
           <visual>
-              <origin xyz="0 0 -0.05"/>
+              <origin xyz="0 0 -0.1"/>
               <geometry>
                   <cylinder radius="0.01" length="0.1"/>
