Commit message: changes

File: src/diffdrive_arduino/description/urdf/diffbot_description.urdf.xacro (robot description, xacro)
@@ -14,4 +14,12 @@
   <xacro:property name="caster_wheel_radius" value="0.015" />
   <xacro:property name="z_offset" value="-${base_height/2}" /> <!-- Space btw top of beam and the each joint -->
+      <!-- BASE_FOOTPRINT LINK -->
+<joint name="base_footprint_joint" type="fixed">
+        <parent link="base_link"/>
+        <child link="base_footprint"/>
+        <origin xyz="0 0 0" rpy="0 0 0"/>
+    </joint>
+    <link name="base_footprint">
+    </link>
   <!-- Base Link -->
   <link name="${prefix}base_link">
